Commit message: Updating with world

File: agri_mapper_simulation/models/rplidar.xacro (robot description, xacro)
@@ -16,4 +16,7 @@
       <sphere radius="0.1" />
     </geometry>
+    <material name="transparent_acrylic">
+      <color rgba="0.0 0.0 0.0 0.4" />
+    </material>
   </visual>
   <collision>
@@ -27,7 +30,6 @@
   <visual>
     <geometry>
-      <sphere radius="0.001" />
+      <sphere radius="0.01" />
     </geometry>
-    <material name="blue" />
   </visual>
   </link>

Commit message: model visible in gazebo Added inertia

File: agri_mapper_simulation/models/rplidar.xacro (robot description, xacro)
@@ -26,4 +26,8 @@
     </geometry>
   </collision>
+  <inertial>
+    <mass value="0.5" />
+    <inertia ixx="0.0" ixy="0.0" ixz="0.0" iyy="0.000001" iyz="0.0" izz="0.0" />
+  </inertial>
   </link>
   <link name="rplidar_frame">

Commit message: Added dependancy

File: agri_mapper_simulation/models/rplidar.xacro (robot description, xacro)
@@ -1,5 +1,5 @@
 <?xml version="1.0"?>
 <robot xmlns:xacro="http://www.ros.org/wiki/xacro" name="rp_lidar">
-  <gazebo>
+  <model name="rp_lidar">
     <plugin name="object_controller" filename="libgazebo_ros_planar_move.so">
       <commandTopic>cmd_vel</commandTopic>
@@ -9,5 +9,5 @@
       <robotBaseFrame>base_link</robotBaseFrame>
     </plugin>
-  </gazebo>
+  </model>
   <link name="base_link">
   <visual>
@@ -16,5 +16,5 @@
       <sphere radius="0.1" />
     </geometry>
-    <material name="transparent_acrylic">
+    <material name="material">
       <color rgba="0.0 0.0 0.0 0.4" />
     </material>
@@ -27,21 +27,10 @@
   </collision>
   <inertial>
-    <mass value="0.5" />
-    <inertia ixx="0.0" ixy="0.0" ixz="0.0" iyy="0.000001" iyz="0.0" izz="0.0" />
+    <mass value="50" />
+    <origin xyz="0 0 -1.25" />
+    <inertia ixx="50.0" ixy="0.0" ixz="0.0" iyy="50.0" iyz="0.0" izz="50.0" />
   </inertial>
   </link>
-  <link name="rplidar_frame">
-  <visual>
-    <geometry>
-      <sphere radius="0.01" />
-    </geometry>
-  </visual>
-  </link>
-  <joint name="base_link_rplidar_frame" type="fixed">
-    <origin xyz="0 0 0" rpy="0 0 0" />
-    <parent link="base_link" />
-    <child link="rplidar_frame" />
-  </joint>
-  <gazebo reference="rplidar_frame">
+  <gazebo reference="base_link">
     <sensor type="ray" name="rplidar_sensor">
       <pose>0 0 0 0 0 0</pose>
@@ -69,6 +58,6 @@
       </ray>
       <plugin name="gazebo_ros_rplidar_controller" filename="libgazebo_ros_laser.so">
-        <topicName>/agri_mapper/scan</topicName>
-        <frameName>/rplidar_frame</frameName>
+        <topicName>/scan</topicName>
+        <frameName>/base_link</frameName>
       </plugin>
     </sensor>
