Commit message: Updated Xacro for wheel and body

File: agri_mapper_description/xacro/bot.xacro (robot description, xacro)
@@ -3,14 +3,14 @@
     <xacro:property name="wheel_center_dist" value="0.31"/>
     <xacro:property name="M_PI" value="3.1415926535897931"/>
-    <xacro:property name="ground_clearance" value="0.203"/>
+    <xacro:property name="ground_clearance" value="0.14"/>
     <link name="base_link"/>
     <link name="chassis_link">
         <visual>
-            <origin xyz="0 1 0" rpy="0 0 0"/>
+            <origin xyz="0.4 0 0" rpy="0 0 0"/>
             <geometry>
-                <box size="0.6 .2 .1"/>
+                <box size="0.9 .5 .1"/>
             </geometry>
             <material name="white">
-                <color rgba="1 1 1 1"/>
+                <color rgba="1 1 1 0.3"/>
             </material>
         </visual>
@@ -21,3 +21,47 @@
         <child link="chassis_link"/>
     </joint>
+    <link name="wheel_l">
+        <visual>
+            <origin xyz="0 0.304 0" rpy="${M_PI/2} 0 0"/>
+            <geometry>
+                <cylinder length="0.05" radius=".14"/>
+            </geometry>
+            <material name="wheel">
+                <color rgba="0 0 1 1"/>
+            </material>
+        </visual>
+        <visual>
+            <origin xyz="0 0.264 0" rpy="${M_PI/2} 0 0"/>
+            <geometry>
+                <cylinder length="0.03" radius=".04"/>
+            </geometry>
+            <material name="wheel"/>
+        </visual>
+    </link>
+    <joint name="chassis_wheel_l" type="fixed">
+        <origin xyz="0 0 0" rpy="0 0 0"/>
+        <parent link="chassis_link"/>
+        <child link="wheel_l"/>
+    </joint>
+    <link name="wheel_r">
+        <visual>
+            <origin xyz="0 -0.304 0" rpy="${-M_PI/2} 0 0"/>
+            <geometry>
+                <cylinder length="0.05" radius=".14"/>
+            </geometry>
+            <material name="wheel"/>
+        </visual>
+        <visual>
+            <origin xyz="0 -0.264 0" rpy="${-M_PI/2} 0 0"/>
+            <geometry>
+                <cylinder length="0.03" radius=".04"/>
+            </geometry>
+            <material name="wheel"/>
+        </visual>
+    </link>
+    <joint name="chassis_wheel_r" type="fixed">
+        <origin xyz="0 0 0" rpy="0 0 0"/>
+        <parent link="chassis_link"/>
+        <child link="wheel_r"/>
+    </joint>
 </robot>

Commit message: Updated bot for continous rotation of wheels

File: agri_mapper_description/xacro/bot.xacro (robot description, xacro)
@@ -39,6 +39,7 @@
         </visual>
     </link>
-    <joint name="chassis_wheel_l" type="fixed">
+    <joint name="chassis_wheel_l" type="continuous">
         <origin xyz="0 0 0" rpy="0 0 0"/>
+        <axis rpy="0 0 0" xyz="0 1 0"/>
         <parent link="chassis_link"/>
         <child link="wheel_l"/>
@@ -60,6 +61,7 @@
         </visual>
     </link>
-    <joint name="chassis_wheel_r" type="fixed">
+    <joint name="chassis_wheel_r" type="continuous">
         <origin xyz="0 0 0" rpy="0 0 0"/>
+        <axis rpy="0 0 0" xyz="0 1 0"/>
         <parent link="chassis_link"/>
         <child link="wheel_r"/>

Commit message: Added RPLidar and Meshes, RVIZ Laser Scan Working Properly

File: agri_mapper_description/xacro/bot.xacro (robot description, xacro)
@@ -1,7 +1,8 @@
 <?xml version="1.0"?>
 <robot name="agri_mapper" xmlns:xacro="http://www.ros.org/wiki/xacro">
-    <xacro:property name="wheel_center_dist" value="0.31"/>
+    <xacro:include filename="$(find agri_mapper_description)/xacro/materials.xacro"/>
     <xacro:property name="M_PI" value="3.1415926535897931"/>
     <xacro:property name="ground_clearance" value="0.14"/>
+    <xacro:property name="rplidar_height" value="0.5"/>
     <link name="base_link"/>
     <link name="chassis_link">
@@ -67,3 +68,89 @@
         <child link="wheel_r"/>
     </joint>
+    <!-- ======================================================= RP lidar Base ====================================================================== -->
+    <link name="lidar_base">
+        <visual>
+            <origin xyz="0.01 0 ${rplidar_height}" rpy="${pi/2} 0 0"/>
+            <geometry>
+                <mesh filename="package://agri_mapper_description/meshes/lidar_base.stl" scale="0.001 0.001 0.001"/>
+            </geometry>
+            <material name="transparent_acrylic_dark"/>
+        </visual>
+    </link>
+    <joint name="chassis_link_lidar_base" type="fixed">
+        <parent link="chassis_link"/>
+        <child link="lidar_base"/>
+    </joint>
+    <!-- ======================================================= RPlidar ====================================================================== -->
+    <link name="lidar_bottom">
+        <visual>
+            <origin xyz="0.0 0 ${rplidar_height + 0.0476}" rpy="${pi/2} 0 0"/>
+            <geometry>
+                <mesh filename="package://agri_mapper_description/meshes/lidar_bottom.stl" scale="0.001 0.001 0.001"/>
+            </geometry>
+            <material name="aluminium"/>
+        </visual>
+    </link>
+    <joint name="lidar_base_lidar_bottom" type="fixed">
+        <parent link="lidar_base"/>
+        <child link="lidar_bottom"/>
+    </joint>
+    <link name="lidar_up">
+        <visual>
+            <origin xyz="0.0 0 ${rplidar_height + 0.0446}" rpy="${pi/2} 0 0"/>
+            <geometry>
+                <mesh filename="package://agri_mapper_description/meshes/lidar_up.stl" scale="0.001 0.001 0.001"/>
+            </geometry>
+            <material name="black_plastic"/>
+        </visual>
+    </link>
+    <joint name="lidar_bottom_lidar_up" type="fixed">
+        <parent link="lidar_bottom"/>
+        <child link="lidar_up"/>
+    </joint>
+    <link name="rplidar_frame">
+        <visual>
+            <geometry>
+                <sphere radius="0.001"/>
+            </geometry>
+            <material name="blue"/>
+        </visual>
+    </link>
+    <joint name="chassis_link_rplidar_frame" type="fixed">
+        <origin xyz="0.0 0 ${rplidar_height + 0.0466}" rpy="0 0 0"/>
+        <parent link="chassis_link"/>
+        <child link="rplidar_frame"/>
+    </joint>
+    <!--
+    <gazebo reference="rplidar_frame">
+        <sensor type="ray" name="rplidar_sensor">
+            <pose>0 0 0 0 0 0</pose>
+            <visualize>true</visualize>
+            <update_rate>8</update_rate>
+            <ray>
+                <scan>
+                    <horizontal>
+                        <samples>360</samples>
+                        <resolution>1</resolution>
+                        <min_angle>0</min_angle>
+                        <max_angle>${pi*2}</max_angle>
+                    </horizontal>
+                </scan>
+                <range>
+                    <min>0.2</min>
+                    <max>6.0</max>
+                    <resolution>0.5</resolution>
+                </range>
+                <noise>
+                    <type>gaussian</type>
+                    <mean>0.0</mean>
+                    <stddev>0.01</stddev>
+                </noise>
+            </ray>
+            <plugin name="gazebo_ros_rplidar_controller" filename="libgazebo_ros_laser.so">
+                <topicName>/lidar_robot/scan</topicName>
+                <frameName>/rplidar_frame</frameName>
+            </plugin>
+        </sensor>
+    </gazebo>-->
 </robot>

Commit message: Updated xacro for showing x and y

File: agri_mapper_description/xacro/bot.xacro (robot description, xacro)
@@ -122,4 +122,34 @@
         <child link="rplidar_frame"/>
     </joint>
+    <link name="x">
+        <visual>
+            <geometry>
+                <sphere radius="0.1"/>
+            </geometry>
+            <material name="x">
+                <color rgba="1.0 0.0 0.0 0.3"/>
+            </material>
+        </visual>
+    </link>
+    <joint name="base_link_x" type="fixed">
+        <origin xyz="1.0 0 0" rpy="0 0 0"/>
+        <parent link="base_link"/>
+        <child link="x"/>
+    </joint>
+    <link name="y">
+        <visual>
+            <geometry>
+                <sphere radius="0.1"/>
+            </geometry>
+            <material name="y">
+                <color rgba="0.0 1.0 0.0 0.3"/>
+            </material>
+        </visual>
+    </link>
+    <joint name="base_link_y" type="fixed">
+        <origin xyz="0 1 0" rpy="0 0 0"/>
+        <parent link="base_link"/>
+        <child link="y"/>
+    </joint>
     <!--
     <gazebo reference="rplidar_frame">

Commit message: Added meshes

File: agri_mapper_description/xacro/bot.xacro (robot description, xacro)
@@ -3,16 +3,13 @@
     <xacro:include filename="$(find agri_mapper_description)/xacro/materials.xacro"/>
     <xacro:property name="M_PI" value="3.1415926535897931"/>
-    <xacro:property name="ground_clearance" value="0.14"/>
+    <xacro:property name="ground_clearance" value="0.07"/>
     <xacro:property name="rplidar_height" value="0.5"/>
     <link name="base_link"/>
     <link name="chassis_link">
         <visual>
-            <origin xyz="0.4 0 0" rpy="0 0 0"/>
+            <origin xyz="-0.67 0.27 0" rpy="${M_PI/2} 0 0"/>
             <geometry>
-                <box size="0.9 .5 .1"/>
+                <mesh filename="package://agri_mapper_description/meshes/frame.stl" scale="0.001 0.001 0.001"/>
             </geometry>
-            <material name="white">
-                <color rgba="1 1 1 0.3"/>
-            </material>
         </visual>
     </link>
@@ -24,18 +21,8 @@
     <link name="wheel_l">
         <visual>
-            <origin xyz="0 0.304 0" rpy="${M_PI/2} 0 0"/>
+            <origin xyz="0.07 0.27 -0.07" rpy="0 0 ${M_PI/2}"/>
             <geometry>
-                <cylinder length="0.05" radius=".14"/>
+                <mesh filename="package://agri_mapper_description/meshes/wheel.stl" scale="0.001 0.001 0.001"/>
             </geometry>
-            <material name="wheel">
-                <color rgba="0 0 1 1"/>
-            </material>
-        </visual>
-        <visual>
-            <origin xyz="0 0.264 0" rpy="${M_PI/2} 0 0"/>
-            <geometry>
-                <cylinder length="0.03" radius=".04"/>
-            </geometry>
-            <material name="wheel"/>
         </visual>
     </link>
@@ -46,4 +33,5 @@
         <child link="wheel_l"/>
     </joint>
+    <!--
     <link name="wheel_r">
         <visual>
@@ -68,5 +56,7 @@
         <child link="wheel_r"/>
     </joint>
+    -->
     <!-- ======================================================= RP lidar Base ====================================================================== -->
+    <!--
     <link name="lidar_base">
         <visual>
@@ -82,5 +72,7 @@
         <child link="lidar_base"/>
     </joint>
+    -->
     <!-- ======================================================= RPlidar ====================================================================== -->
+    <!--
     <link name="lidar_bottom">
         <visual>
@@ -152,4 +144,5 @@
         <child link="y"/>
     </joint>
+    -->
     <!--
     <gazebo reference="rplidar_frame">

Commit message: Updated model

File: agri_mapper_description/xacro/bot.xacro (robot description, xacro)
@@ -8,5 +8,5 @@
     <link name="chassis_link">
         <visual>
-            <origin xyz="-0.67 0.27 0" rpy="${M_PI/2} 0 0"/>
+            <origin xyz="0 0 0" rpy="${M_PI/2} 0 0"/>
             <geometry>
                 <mesh filename="package://agri_mapper_description/meshes/frame.stl" scale="0.001 0.001 0.001"/>
@@ -21,5 +21,5 @@
     <link name="wheel_l">
         <visual>
-            <origin xyz="0.07 0.27 -0.07" rpy="0 0 ${M_PI/2}"/>
+            <origin xyz="0 0.27 0" rpy="0 0 ${M_PI/2}"/>
             <geometry>
                 <mesh filename="package://agri_mapper_description/meshes/wheel.stl" scale="0.001 0.001 0.001"/>
@@ -33,19 +33,10 @@
         <child link="wheel_l"/>
     </joint>
-    <!--
     <link name="wheel_r">
         <visual>
-            <origin xyz="0 -0.304 0" rpy="${-M_PI/2} 0 0"/>
+            <origin xyz="0 -0.27 0" rpy="0 0 ${M_PI/2}"/>
             <geometry>
-                <cylinder length="0.05" radius=".14"/>
+                <mesh filename="package://agri_mapper_description/meshes/wheel.stl" scale="0.001 0.001 0.001"/>
             </geometry>
-            <material name="wheel"/>
-        </visual>
-        <visual>
-            <origin xyz="0 -0.264 0" rpy="${-M_PI/2} 0 0"/>
-            <geometry>
-                <cylinder length="0.03" radius=".04"/>
-            </geometry>
-            <material name="wheel"/>
         </visual>
     </link>
@@ -56,5 +47,4 @@
         <child link="wheel_r"/>
     </joint>
-    -->
     <!-- ======================================================= RP lidar Base ====================================================================== -->
     <!--

Commit message: Completed Model

File: agri_mapper_description/xacro/bot.xacro (robot description, xacro)
@@ -4,16 +4,18 @@
     <xacro:property name="M_PI" value="3.1415926535897931"/>
     <xacro:property name="ground_clearance" value="0.07"/>
-    <xacro:property name="rplidar_height" value="0.5"/>
+    <xacro:property name="stand_to_rplidar_height" value="0.1"/>
+    <xacro:property name="stand_height" value="0.772"/>
+    <xacro:property name="scale" value="0.001"/>
     <link name="base_link"/>
     <link name="chassis_link">
         <visual>
-            <origin xyz="0 0 0" rpy="${M_PI/2} 0 0"/>
-            <geometry>
-                <mesh filename="package://agri_mapper_description/meshes/frame.stl" scale="0.001 0.001 0.001"/>
-            </geometry>
+            <geometry>
+                <mesh filename="package://agri_mapper_description/meshes/frame.stl" scale="${scale} ${scale} ${scale}"/>
+            </geometry>
+            <material name="grey"/>
         </visual>
     </link>
     <joint name="chassis_joint" type="fixed">
-        <origin xyz="0 0 ${ground_clearance}" rpy="0 0 0"/>
+        <origin xyz="0 0 ${ground_clearance}" rpy="${M_PI/2} 0 ${M_PI}"/>
         <parent link="base_link"/>
         <child link="chassis_link"/>
@@ -21,37 +23,50 @@
     <link name="wheel_l">
         <visual>
-            <origin xyz="0 0.27 0" rpy="0 0 ${M_PI/2}"/>
-            <geometry>
-                <mesh filename="package://agri_mapper_description/meshes/wheel.stl" scale="0.001 0.001 0.001"/>
-            </geometry>
+            <geometry>
+                <mesh filename="package://agri_mapper_description/meshes/wheel.stl" scale="${scale} ${scale} ${scale}"/>
+            </geometry>
+            <material name="black"/>
         </visual>
     </link>
     <joint name="chassis_wheel_l" type="continuous">
-        <origin xyz="0 0 0" rpy="0 0 0"/>
+        <origin xyz="0 0 0.27" rpy="0 ${-M_PI/2} 0"/>
+        <axis rpy="0 0 0" xyz="1 0 0"/>
+        <parent link="chassis_link"/>
+        <child link="wheel_l"/>
+    </joint>
+    <link name="wheel_r">
+        <visual>
+            <geometry>
+                <mesh filename="package://agri_mapper_description/meshes/wheel.stl" scale="${scale} ${scale} ${scale}"/>
+            </geometry>
+            <material name="black"/>
+        </visual>
+    </link>
+    <joint name="chassis_wheel_r" type="continuous">
+        <origin xyz="0 0 -0.27" rpy="0 ${-M_PI/2} 0"/>
+        <axis rpy="0 0 0" xyz="1 0 0"/>
+        <parent link="chassis_link"/>
+        <child link="wheel_r"/>
+    </joint>
+    <link name="lidar_stand">
+        <visual>
+            <geometry>
+                <mesh filename="package://agri_mapper_description/meshes/lidar_stand.stl" scale="${scale} ${scale} ${scale}"/>
+            </geometry>
+            <material name="black"/>
+        </visual>
+    </link>
+    <joint name="chassis_lidar_stand" type="prismatic">
+        <origin xyz="0 ${stand_height} 0" rpy="0 ${M_PI/2} 0"/>
         <axis rpy="0 0 0" xyz="0 1 0"/>
         <parent link="chassis_link"/>
-        <child link="wheel_l"/>
-    </joint>
-    <link name="wheel_r">
-        <visual>
-            <origin xyz="0 -0.27 0" rpy="0 0 ${M_PI/2}"/>
-            <geometry>
-                <mesh filename="package://agri_mapper_description/meshes/wheel.stl" scale="0.001 0.001 0.001"/>
-            </geometry>
-        </visual>
-    </link>
-    <joint name="chassis_wheel_r" type="continuous">
-        <origin xyz="0 0 0" rpy="0 0 0"/>
-        <axis rpy="0 0 0" xyz="0 1 0"/>
-        <parent link="chassis_link"/>
-        <child link="wheel_r"/>
-    </joint>
-    <!-- ======================================================= RP lidar Base ====================================================================== -->
-    <!--
+        <child link="lidar_stand"/>
+        <limit effort="50.0" velocity="0.2" lower="0" upper="0.338"/>
+    </joint>
+    <!-- ===================================== RP lidar Base ======================================= -->
     <link name="lidar_base">
         <visual>
-            <origin xyz="0.01 0 ${rplidar_height}" rpy="${pi/2} 0 0"/>
-            <geometry>
-                <mesh filename="package://agri_mapper_description/meshes/lidar_base.stl" scale="0.001 0.001 0.001"/>
+            <geometry>
+                <mesh filename="package://agri_mapper_description/meshes/lidar_base.stl" scale="${scale} ${scale} ${scale}"/>
             </geometry>
             <material name="transparent_acrylic_dark"/>
@@ -59,15 +74,13 @@
     </link>
     <joint name="chassis_link_lidar_base" type="fixed">
-        <parent link="chassis_link"/>
+        <origin xyz="0 ${stand_to_rplidar_height} -0.01" rpy="0 ${M_PI/2} 0"/>
+        <parent link="lidar_stand"/>
         <child link="lidar_base"/>
     </joint>
-    -->
-    <!-- ======================================================= RPlidar ====================================================================== -->
-    <!--
+    <!-- ======================================= RPlidar ============================================== -->
     <link name="lidar_bottom">
         <visual>
-            <origin xyz="0.0 0 ${rplidar_height + 0.0476}" rpy="${pi/2} 0 0"/>
-            <geometry>
-                <mesh filename="package://agri_mapper_description/meshes/lidar_bottom.stl" scale="0.001 0.001 0.001"/>
+            <geometry>
+                <mesh filename="package://agri_mapper_description/meshes/lidar_bottom.stl" scale="${scale} ${scale} ${scale}"/>
             </geometry>
             <material name="aluminium"/>
@@ -75,4 +88,5 @@
     </link>
     <joint name="lidar_base_lidar_bottom" type="fixed">
+        <origin xyz="-0.01 0.0476 0" rpy="0 0 0"/>
         <parent link="lidar_base"/>
         <child link="lidar_bottom"/>
@@ -80,7 +94,6 @@
     <link name="lidar_up">
         <visual>
-            <origin xyz="0.0 0 ${rplidar_height + 0.0446}" rpy="${pi/2} 0 0"/>
-            <geometry>
-                <mesh filename="package://agri_mapper_description/meshes/lidar_up.stl" scale="0.001 0.001 0.001"/>
+            <geometry>
+                <mesh filename="package://agri_mapper_description/meshes/lidar_up.stl" scale="${scale} ${scale} ${scale}"/>
             </geometry>
             <material name="black_plastic"/>
@@ -88,4 +101,5 @@
     </link>
     <joint name="lidar_bottom_lidar_up" type="fixed">
+        <origin xyz="0 0 0" rpy="0 0 0"/>
         <parent link="lidar_bottom"/>
         <child link="lidar_up"/>
@@ -94,14 +108,15 @@
         <visual>
             <geometry>
-                <sphere radius="0.001"/>
-            </geometry>
-            <material name="blue"/>
+                <sphere radius="0.02"/>
+            </geometry>
+            <material name="red"/>
         </visual>
     </link>
     <joint name="chassis_link_rplidar_frame" type="fixed">
-        <origin xyz="0.0 0 ${rplidar_height + 0.0466}" rpy="0 0 0"/>
-        <parent link="chassis_link"/>
+        <origin xyz="0 0 0.001" rpy="0 0 0"/>
+        <parent link="lidar_up"/>
         <child link="rplidar_frame"/>
     </joint>
+    <!-- ======================================= References ============================================== -->
     <link name="x">
         <visual>
@@ -133,4 +148,20 @@
         <parent link="base_link"/>
         <child link="y"/>
+    </joint>
+    <!--
+    <link name="z">
+        <visual>
+            <origin xyz="0 0 0" rpy="0 0 0"/>
+            <geometry>
+                <cylinder radius="0.002" length="3"/>
+            </geometry>
+            <material name="z">
+                <color rgba="0.0 0.0 1.0 1"/>
+            </material>
+        </visual>
+    </link>
+    <joint name="base_link_z" type="fixed">
+        <parent link="base_link"/>
+        <child link="z"/>
     </joint>
     -->

Commit message: Solved orientation of lidar_frame

File: agri_mapper_description/xacro/bot.xacro (robot description, xacro)
@@ -113,6 +113,6 @@
         </visual>
     </link>
-    <joint name="chassis_link_rplidar_frame" type="fixed">
-        <origin xyz="0 0 0.001" rpy="0 0 0"/>
+    <joint name="lidar_up_rplidar_frame" type="fixed">
+        <origin xyz="0 0 0.001" rpy="${pi/2} ${pi} ${pi}"/>
         <parent link="lidar_up"/>
         <child link="rplidar_frame"/>
